File: PROJECT.kicad_pcb (KiCad board)
At the start: 2 copper layers, 133.4 x 95.4 mm, 95 parts, among them J1 Conn_01x04, Q1 SI2302, Q2 SI2302, U1 Core51822B, k1 KEYSW

Commit message: Pcb
Parts:
- moved D11 5.57 mm to (106.3, 80.4)
Routing:
- net VCC: track 202.0 -> 0.00 mm, vias 5 -> 0
- net GND_BAT: track 190.3 -> 0.00 mm
- net ROW4: track 231.3 -> 88.2 mm, vias 2 -> 0
- net VCC_S: track 93.5 -> 0.00 mm, vias 3 -> 0
- net ROW3: track 219.8 -> 130.6 mm, vias 6 -> 0
- net ROW2: track 205.3 -> 123.4 mm, vias 4 -> 0
- net COL6: track 151.6 -> 79.5 mm, vias 1 -> 0
- net COL0: track 125.4 -> 77.6 mm
- net SWCLK: track 47.2 -> 0.00 mm
- net COL5: track 126.5 -> 79.4 mm, vias 1 -> 0
- net SWDIO: track 46.7 -> 0.00 mm
- net ROW1: track 171.6 -> 130.8 mm
- net (no net): track 0.00 -> 39.6 mm
- net ROW0: track 162.5 -> 124.4 mm
- net COL1: track 119.0 -> 82.5 mm, vias 2 -> 0
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
Commit message: Re-routed
Parts:
- moved D9 9.69 mm to (80.9, 80.9)
- moved D8 9.25 mm to (60.3, 81.0)
- moved D32 6.16 mm to (123.5, 134.0)
- moved D30 5.85 mm to (85.1, 133.9)
- moved D10 5.46 mm to (87.1, 80.9)
- moved D29 2.34 mm to (66.5, 133.9)
- moved D31 2.25 mm to (104.5, 134.1)
- moved D4 1.53 mm to (123.3, 59.3)
- moved D11 0.94 mm to (107.0, 81.0)
- moved D1 0.89 mm to (63.7, 51.4), turned to 270 degrees
- moved D2 0.79 mm to (82.9, 51.6), turned to 270 degrees
Routing:
- net VCC: track 0.00 -> 166.3 mm, vias 0 -> 4
- net GND_BAT: track 0.00 -> 165.8 mm, vias 0 -> 4
- net ROW4: track 88.2 -> 207.6 mm, vias 0 -> 2
- net VCC_S: track 0.00 -> 101.3 mm, vias 0 -> 1
- net ROW3: track 130.6 -> 215.1 mm, vias 0 -> 2
- net COL6: track 79.5 -> 162.6 mm, vias 0 -> 1
- net ROW2: track 123.4 -> 194.5 mm, vias 0 -> 2
- net COL5: track 79.4 -> 134.3 mm, vias 0 -> 1
- net SWCLK: track 0.00 -> 47.2 mm
- net SWDIO: track 0.00 -> 46.7 mm
- net COL0: track 77.6 -> 123.6 mm
- net (no net): track 39.6 -> 0.00 mm
- net ROW1: track 130.8 -> 162.1 mm, vias 0 -> 2
- net COL1: track 82.5 -> 112.2 mm
- net ROW0: track 124.4 -> 148.1 mm
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