File: PROJECT.kicad_pcb (KiCad board)
At the start: 2 copper layers, 133.4 x 95.4 mm, 95 parts, among them J1 Conn_01x04, Q1 SI2302, Q2 SI2302, U1 Core51822B, k1 KEYSW

Commit message: Re-routed
Parts:
- removed the P? at (162.0, 66.3)
- removed the P? at (142.9, 66.3)
- removed the P? at (66.8, 123.9)
- removed the P? at (105.5, 123.8)
- removed the P? at (142.9, 124.0)
- removed the P? at (161.8, 123.9)
- added G***: LOGO, Mixed Lib:Medusa, F.Cu at (114.0, 91.7)
- moved D9 9.69 mm to (80.9, 80.9)
- moved D8 9.25 mm to (60.3, 81.0)
- moved D32 6.16 mm to (123.5, 134.0)
- moved D30 5.85 mm to (85.1, 133.9)
- moved D10 5.46 mm to (87.1, 80.9)
- moved D29 2.34 mm to (66.5, 133.9)
- moved D31 2.25 mm to (104.5, 134.1)
- moved D4 1.53 mm to (123.3, 59.3)
- moved D11 0.94 mm to (107.0, 81.0)
- moved D1 0.89 mm to (63.7, 51.4), turned to 270 degrees
- moved D2 0.79 mm to (82.9, 51.6), turned to 270 degrees
Routing:
- net VCC: track 0.00 -> 166.3 mm, vias 0 -> 4
- net GND_BAT: track 0.00 -> 165.8 mm, vias 0 -> 4
- net ROW4: track 88.2 -> 207.6 mm, vias 0 -> 2
- net VCC_S: track 0.00 -> 101.3 mm, vias 0 -> 1
- net ROW3: track 130.6 -> 215.1 mm, vias 0 -> 2
- net COL6: track 79.5 -> 162.6 mm, vias 0 -> 1
- net ROW2: track 123.4 -> 194.5 mm, vias 0 -> 2
- net COL5: track 79.4 -> 134.3 mm, vias 0 -> 1
- net SWCLK: track 0.00 -> 47.2 mm
- net SWDIO: track 0.00 -> 46.7 mm
- net COL0: track 77.6 -> 123.6 mm
- net (no net): track 39.6 -> 0.00 mm
- net ROW1: track 130.8 -> 162.1 mm, vias 0 -> 2
- net COL1: track 82.5 -> 112.2 mm
- net ROW0: track 124.4 -> 148.1 mm
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Other:
- outline, holes or cut-outs redrawn
- board text added: "GND"
- board text added: "JLCJLCJLCJLC"
- board text added: "SWCLK"
- board text added: "SWDIO"
- board text added: "VCC"
- board text added: "Ver 1.0"
