File: PROJECT.kicad_pcb (KiCad board)
At the start: 2 copper layers, 133.4 x 95.4 mm, 90 parts, among them J1 Conn_01x04, Q1 SI2302, Q2 SI2302, U1 Core51822B, k1 KEYSW

Commit message: Plate design
Parts:
- moved J1 1.87 mm to (49.0, 68.3)
Routing:
- net VCC: track 166.3 -> 168.2 mm, vias 4 -> 5
- net SWDIO: track 46.7 -> 48.5 mm
- net SWCLK: track 47.2 -> 49.1 mm
- net GND: vias 28 -> 29
Changed lines of the file:
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@@
     (thickness 1.6)
     (drawings 146)
-    (tracks 568)
+    (tracks 573)
     (zones 0)
     (modules 90)
@@
     (38 B.Mask user)
     (39 F.Mask user)
-    (40 Dwgs.User user hide)
+    (40 Dwgs.User user)
     (41 Cmts.User user hide)
     (42 Eco1.User user)
@@
   )
   (module mitosis-parts:programming_port (layer B.Cu)
-    (at 50.92192 68.33108 180)
+    (at 49.04994 68.326 180)
     (fp_text reference J1 (at -0.08128 -2.02692 180) (layer B.SilkS)
       (effects (font (size 1 1) (thickness 0.15)) (justify mirror))
@@
   (segment (start 103.5685 116.0145) (end 104.79024 117.23624) (width 0.3556) (layer F.Cu) (net 2))
   (segment (start 104.79024 117.23624) (end 104.79024 119.41436) (width 0.3556) (layer F.Cu) (net 2))
-  (segment (start 50.92192 65.79108) (end 49.68748 67.02552) (width 0.3556) (layer B.Cu) (net 2))
-  (segment (start 49.68748 67.02552) (end 49.68748 69.68236) (width 0.3556) (layer B.Cu) (net 2))
-  (segment (start 49.68748 69.68236) (end 50.165 70.15988) (width 0.3556) (layer B.Cu) (net 2))
   (segment (start 81.28 110.2096) (end 81.28 100.52404) (width 0.3556) (layer B.Cu) (net 2))
-  (segment (start 50.165 70.15988) (end 50.165 72.97928) (width 0.3556) (layer B.Cu) (net 2))
-  (segment (start 50.165 72.97928) (end 50.17008 72.98436) (width 0.3556) (layer B.Cu) (net 2))
-  (segment (start 50.570842 86.77148) (end 52.668882 88.86952) (width 0.3556) (layer B.Cu) (net 2))
-  (segment (start 52.668882 88.86952) (end 53.14188 88.86952) (width 0.3556) (layer B.Cu) (net 2))
-  (segment (start 53.14188 88.86952) (end 56.57596 92.3036) (width 0.3556) (layer B.Cu) (net 2))
-  (segment (start 56.57596 92.3036) (end 68.76288 92.3036) (width 0.3556) (layer B.Cu) (net 2))
-  (segment (start 68.76288 92.3036) (end 75.1078 98.64852) (width 0.3556) (layer B.Cu) (net 2))
-  (segment (start 79.40448 98.64852) (end 81.28 100.52404) (width 0.3556) (layer B.Cu) (net 2))
-  (segment (start 75.1078 98.64852) (end 79.40448 98.64852) (width 0.3556) (layer B.Cu) (net 2))
+  (segment (start 50.165 66.90106) (end 49.04994 65.786) (width 0.3556) (layer B.Cu) (net 2))
+  (segment (start 50.165 72.97928) (end 50.165 66.90106) (width 0.3556) (layer B.Cu) (net 2))
+  (segment (start 50.17008 86.34984) (end 50.17008 72.98436) (width 0.3556) (layer B.Cu) (net 2))
   (segment (start 50.570842 86.750602) (end 50.17008 86.34984) (width 0.3556) (layer B.Cu) (net 2))
   (segment (start 50.570842 86.77148) (end 50.570842 86.750602) (width 0.3556) (layer B.Cu) (net 2))
-  (segment (start 50.17008 72.98436) (end 50.17008 86.34984) (width 0.3556) (layer B.Cu) (net 2))
+  (segment (start 50.17008 72.98436) (end 50.165 72.97928) (width 0.3556) (layer B.Cu) (net 2))
+  (segment (start 81.28 100.52404) (end 79.40448 98.64852) (width 0.3556) (layer B.Cu) (net 2))
+  (segment (start 75.1078 98.64852) (end 68.76288 92.3036) (width 0.3556) (layer B.Cu) (net 2))
+  (segment (start 52.668882 88.86952) (end 50.570842 86.77148) (width 0.3556) (layer B.Cu) (net 2))
+  (segment (start 68.76288 92.3036) (end 56.57596 92.3036) (width 0.3556) (layer B.Cu) (net 2))
+  (segment (start 79.40448 98.64852) (end 75.1078 98.64852) (width 0.3556) (layer B.Cu) (net 2))
+  (segment (start 56.57596 92.3036) (end 53.14188 88.86952) (width 0.3556) (layer B.Cu) (net 2))
+  (segment (start 53.14188 88.86952) (end 52.668882 88.86952) (width 0.3556) (layer B.Cu) (net 2))
   (segment (start 60.085 53.085) (end 63.6905 53.085) (width 0.2032) (layer B.Cu) (net 3))
   (segment (start 59.65 52.65) (end 60.085 53.085) (width 0.2032) (layer B.Cu) (net 3))
@@
   (segment (start 72.201 66.105) (end 68.597081 62.501081) (width 0.2032) (layer B.Cu) (net 43))
   (segment (start 95.775 66.105) (end 72.201 66.105) (width 0.2032) (layer B.Cu) (net 43))
+  (segment (start 50.91684 63.246) (end 49.04994 63.246) (width 0.2032) (layer B.Cu) (net 43))
+  (segment (start 50.92192 63.25108) (end 50.91684 63.246) (width 0.2032) (layer B.Cu) (net 43))
   (via (at 87.884 87.3125) (size 0.6) (drill 0.4) (layers F.Cu B.Cu) (net 44))
   (segment (start 87.884 98.20064) (end 86.802 99.28264) (width 0.3556) (layer F.Cu) (net 44))
@@
   (segment (start 89.68232 87.80272) (end 117.795109 87.80272) (width 0.3556) (layer B.Cu) (net 44))
   (segment (start 121.539 86.741) (end 118.85168 86.746149) (width 0.3556) (layer B.Cu) (net 44))
+  (via (at 50.92192 68.33108) (size 0.6) (drill 0.4) (layers F.Cu B.Cu) (net 44))
+  (segment (start 49.05502 68.33108) (end 49.04994 68.326) (width 0.3556) (layer F.Cu) (net 44))
+  (segment (start 50.92192 68.33108) (end 49.05502 68.33108) (width 0.3556) (layer F.Cu) (net 44))
   (segment (start 53.34 54.61) (end 53.34 73.66) (width 0.2032) (layer F.Cu) (net 45))
   (segment (start 54.274999 96.625001) (end 53.15 97.75) (width 0.2032) (layer F.Cu) (net 45))
@@
   (via (at 59.87796 89.9922) (size 0.6) (drill 0.4) (layers F.Cu B.Cu) (net 52))
   (via (at 51.22672 83.03768) (size 0.6) (drill 0.4) (layers F.Cu B.Cu) (net 52))
-  (segment (start 51.671919 61.461079) (end 51.682079 61.461079) (width 0.2032) (layer B.Cu) (net 53))
-  (segment (start 50.92192 60.71108) (end 51.671919 61.461079) (width 0.2032) (layer B.Cu) (net 53))
-  (segment (start 51.682079 61.461079) (end 52.36464 62.14364) (width 0.2032) (layer B.Cu) (net 53))
-  (segment (start 52.36464 62.14364) (end 68.74764 62.14364) (width 0.2032) (layer B.Cu) (net 53))
-  (segment (start 68.74764 62.14364) (end 72.34936 65.74536) (width 0.2032) (layer B.Cu) (net 53))
-  (segment (start 72.34936 65.74536) (end 93.03512 65.74536) (width 0.2032) (layer B.Cu) (net 53))
-  (segment (start 93.77548 65.005) (end 95.775 65.005) (width 0.2032) (layer B.Cu) (net 53))
-  (segment (start 93.03512 65.74536) (end 93.77548 65.005) (width 0.2032) (layer B.Cu) (net 53))
+  (via (at 132.0673 138.80338) (size 0.6) (drill 0.4) (layers F.Cu B.Cu) (net 52))
+  (segment (start 50.91684 60.706) (end 49.04994 60.706) (width 0.2032) (layer B.Cu) (net 53))
+  (segment (start 51.682079 61.461079) (end 51.671919 61.461079) (width 0.2032) (layer B.Cu) (net 53))
+  (segment (start 93.77548 65.005) (end 93.03512 65.74536) (width 0.2032) (layer B.Cu) (net 53))
+  (segment (start 95.775 65.005) (end 93.77548 65.005) (width 0.2032) (layer B.Cu) (net 53))
+  (segment (start 51.671919 61.461079) (end 50.91684 60.706) (width 0.2032) (layer B.Cu) (net 53))
+  (segment (start 93.03512 65.74536) (end 72.34936 65.74536) (width 0.2032) (layer B.Cu) (net 53))
+  (segment (start 72.34936 65.74536) (end 68.74764 62.14364) (width 0.2032) (layer B.Cu) (net 53))
+  (segment (start 68.74764 62.14364) (end 52.36464 62.14364) (width 0.2032) (layer B.Cu) (net 53))
+  (segment (start 52.36464 62.14364) (end 51.682079 61.461079) (width 0.2032) (layer B.Cu) (net 53))
   (zone (net 52) (net_name GND) (layer B.Cu) (hatch edge 0.508)
     (connect_pads (clearance 0.508))
